File: eagle/remote/pcbremote.sch (EAGLE design)
At the start: 32 parts, among them Q1 FDC638P, U2 ATMEGA328P_TQFP, U3 LTC1540CS8PBF, U4 MCP73831/OT, U5 LTC4412ES6TRPBF, U6 MIC5301-3.3YD5-TR, Y2 8MHz

Commit message: Add Remote Shape
Parts:
- removed LED_EXT_CON: FEMALE 1x2, SparkFun-Retired:CONN_02
- added LED_EXT: JST-XH-02-PIN-ROUND-PAD, Rembrandt Electronics - JST XH Connectors v1-0:JST-XH-02-PIN-ROUND-PAD
- added OLED_CONN: JST-XH-04-PIN-ROUND-PAD, Rembrandt Electronics - JST XH Connectors v1-0:JST-XH-04-PIN-ROUND-PAD
Connections:
- net 3.3V: now also OLED_CONN-2.S
- net GND: now also OLED_CONN-1.S
- net N$5: now also LED_EXT-1.S; no longer LED_EXT_CON.1
- net SCL: now also OLED_CONN-3.S
- net SDA: now also OLED_CONN-4.S
- net V_USB: now also LED_EXT-2.S; no longer LED_EXT_CON.2
Changed lines of the file:
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@@
 <part name="C2" library="rcl" library_urn="urn:adsk.eagle:library:334" deviceset="C-US" device="C0805" package3d_urn="urn:adsk.eagle:package:23617/2" value=".1u"/>
 <part name="SUPPLY15" library="SparkFun-PowerSymbols" deviceset="VIN" device=""/>
-<part name="LED_EXT_CON" library="SparkFun-Retired" deviceset="CONN_02" device="" value="FEMALE 1x2"/>
 <part name="U3" library="LTC_1450" deviceset="LTC1540CS8PBF" device=""/>
 <part name="GND11" library="SparkFun-PowerSymbols" deviceset="GND" device=""/>
@@
 <part name="Q1" library="FDC638P" deviceset="FDC638P" device=""/>
 <part name="D1" library="adafruit" deviceset="DIODE" device="SOD-123"/>
+<part name="LED_EXT" library="Rembrandt Electronics - JST XH Connectors v1-0" deviceset="JST-XH-02-PIN" device="-ROUND-PAD"/>
+<part name="OLED_CONN" library="Rembrandt Electronics - JST XH Connectors v1-0" deviceset="JST-XH-04-PIN" device="-ROUND-PAD"/>
+<part name="GND17" library="SparkFun-PowerSymbols" deviceset="GND" device=""/>
+<part name="SUPPLY9" library="SparkFun-PowerSymbols" deviceset="3.3V" device=""/>
 </parts>
 <sheets>
@@
 <attribute name="VALUE" x="93.98" y="178.308" size="1.778" layer="96" align="bottom-center"/>
 </instance>
-<instance part="LED_EXT_CON" gate="G$1" x="210.82" y="91.44" smashed="yes" grouprefs="LIPO_CHARGING">
-<attribute name="VALUE" x="208.28" y="86.614" size="1.778" layer="96" font="vector"/>
-<attribute name="NAME" x="208.28" y="97.028" size="1.778" layer="95" font="vector"/>
-</instance>
 <instance part="U3" gate="A" x="93.98" y="91.44" smashed="yes" grouprefs="VOLTAGE_MONITOR">
 <attribute name="NAME" x="109.5756" y="100.5586" size="2.0828" layer="95" ratio="6" rot="SR0"/>
@@
 <attribute name="NAME" x="149.86" y="241.3" size="1.27" layer="95"/>
 <attribute name="VALUE" x="149.86" y="234.95" size="1.27" layer="96"/>
+</instance>
+<instance part="LED_EXT" gate="-2" x="215.9" y="93.98" smashed="yes" rot="R180">
+<attribute name="NAME" x="213.36" y="94.742" size="1.524" layer="95" rot="R180"/>
+</instance>
+<instance part="LED_EXT" gate="-1" x="215.9" y="91.44" smashed="yes" rot="R180">
+<attribute name="NAME" x="213.36" y="92.202" size="1.524" layer="95" rot="R180"/>
+<attribute name="VALUE" x="229.362" y="90.043" size="1.778" layer="96" rot="R180"/>
+</instance>
+<instance part="OLED_CONN" gate="-1" x="68.58" y="134.62" smashed="yes">
+<attribute name="NAME" x="71.12" y="133.858" size="1.524" layer="95"/>
+<attribute name="VALUE" x="67.818" y="136.017" size="1.778" layer="96"/>
+</instance>
+<instance part="OLED_CONN" gate="-2" x="68.58" y="132.08" smashed="yes">
+<attribute name="NAME" x="71.12" y="131.318" size="1.524" layer="95"/>
+</instance>
+<instance part="OLED_CONN" gate="-3" x="68.58" y="129.54" smashed="yes">
+<attribute name="NAME" x="71.12" y="128.778" size="1.524" layer="95"/>
+</instance>
+<instance part="OLED_CONN" gate="-4" x="68.58" y="127" smashed="yes">
+<attribute name="NAME" x="71.12" y="126.238" size="1.524" layer="95"/>
+</instance>
+<instance part="GND17" gate="1" x="40.64" y="132.08" smashed="yes">
+<attribute name="VALUE" x="40.64" y="131.826" size="1.778" layer="96" align="top-center"/>
+</instance>
+<instance part="SUPPLY9" gate="G$1" x="60.96" y="132.08" smashed="yes" rot="R90">
+<attribute name="VALUE" x="54.61" y="132.588" size="1.778" layer="96" rot="R180" align="bottom-center"/>
 </instance>
 </instances>
@@
 <junction x="109.22" y="218.44"/>
 </segment>
+<segment>
+<pinref part="OLED_CONN" gate="-1" pin="S"/>
+<pinref part="GND17" gate="1" pin="GND"/>
+<wire x1="66.04" y1="134.62" x2="40.64" y2="134.62" width="0.1524" layer="91"/>
+</segment>
 </net>
 <net name="V_BATT" class="0">
@@
 <wire x1="220.98" y1="104.14" x2="220.98" y2="101.6" width="0.1524" layer="91" grouprefs="LIPO_CHARGING"/>
 <wire x1="220.98" y1="101.6" x2="236.22" y2="101.6" width="0.1524" layer="91" grouprefs="LIPO_CHARGING"/>
-<pinref part="LED_EXT_CON" gate="G$1" pin="2"/>
 <wire x1="236.22" y1="101.6" x2="241.3" y2="101.6" width="0.1524" layer="91" grouprefs="LIPO_CHARGING"/>
 <wire x1="220.98" y1="101.6" x2="220.98" y2="93.98" width="0.1524" layer="91" grouprefs="LIPO_CHARGING"/>
@@
 <wire x1="200.66" y1="101.6" x2="220.98" y2="101.6" width="0.1524" layer="91" grouprefs="LIPO_CHARGING"/>
 <pinref part="USB_IN" gate="G$1" pin="2"/>
+<pinref part="LED_EXT" gate="-2" pin="S"/>
 </segment>
 <segment>
@@
 <junction x="281.94" y="167.64"/>
 </segment>
+<segment>
+<pinref part="OLED_CONN" gate="-2" pin="S"/>
+<pinref part="SUPPLY9" gate="G$1" pin="3.3V"/>
+<wire x1="66.04" y1="132.08" x2="60.96" y2="132.08" width="0.1524" layer="91"/>
+</segment>
 </net>
 <net name="MISO" class="0">
@@
 <pinref part="U2" gate="U1" pin="PC4(ADC4/SDA)"/>
 </segment>
+<segment>
+<pinref part="OLED_CONN" gate="-4" pin="S"/>
+<wire x1="66.04" y1="127" x2="60.96" y2="127" width="0.1524" layer="91"/>
+<label x="54.356" y="126.238" size="1.778" layer="95"/>
+</segment>
 </net>
 <net name="SCL" class="0">
@@
 <label x="272.542" y="172.72" size="1.778" layer="95" grouprefs="ATMEGA328P"/>
 <pinref part="U2" gate="U1" pin="PC5(ADC5/SCL)"/>
+</segment>
+<segment>
+<pinref part="OLED_CONN" gate="-3" pin="S"/>
+<wire x1="66.04" y1="129.54" x2="60.96" y2="129.54" width="0.1524" layer="91"/>
+<label x="55.118" y="128.778" size="1.778" layer="95"/>
 </segment>
 </net>
@@
 <net name="N$5" class="0">
 <segment>
-<pinref part="LED_EXT_CON" gate="G$1" pin="1"/>
 <pinref part="R6" gate="G$1" pin="2"/>
 <wire x1="218.44" y1="91.44" x2="220.98" y2="91.44" width="0.1524" layer="91" grouprefs="LIPO_CHARGING"/>
-</segment>
-</net>
+<pinref part="LED_EXT" gate="-1" pin="S"/>
+</segment>
+</net>

Commit message: Snapped to grid
Parts:
- removed R2: 2.26Meg, rcl:R-US_R0805
- removed R3: 0, rcl:R-US_R0805
- removed R4: 1.18Meg, rcl:R-US_R0805
- added HALL, TRIGGER: JST-XH-02-PIN-ROUND-PAD, Rembrandt Electronics - JST XH Connectors v1-0:JST-XH-02-PIN-ROUND-PAD
- added MASTER_SW, UART: 455-1750-1-ND, SparkFun-Connectors:CONN_03
- added R10, R11: 10k, rcl:R-US_R0805
- added VR1: 3296W-1-502, 3296W-1-502:3296W-1-502
Connections:
- removed net N$2: R2.1, R3.1
- new net N$10: CONN_BAT.1, MASTER_SW.2
- net A2: now also R10.1, R11.2
- net A3: now also HALL-2.S
- net D0: now also UART.2
- net D1: now also UART.3
- net D2: now also TRIGGER-2.S
- net GND: now also HALL-1.S, R11.1, TRIGGER-1.S, UART.1, VR1.CW; no longer R4.1
- net N$1: now also VR1.WIPER; no longer R2.2, R4.2
- net VIN: now also VR1.CCW; no longer R3.2
- net V_BATT: now also MASTER_SW.1, R10.2; no longer CONN_BAT.1
