File: eagle/remote/pcbremote.brd (EAGLE design)
At the start: 37.7 x 83 mm, 39 parts, among them CN1 SOCKET 1x2, IC1 MCP73831/OT, J1 FEMALE 1x2, J2 455-1750-1-ND, J4 FEMALE 2x4, J5 FEMALE 2x3, J6 455-1750-1-ND, Q1 FDC638P, U1 LTC1540CS8PBF, U2 LTC4412ES6TRPBF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

Commit message: Update Hall 3 pin
Parts:
- X4: value JST-XH-02-PIN-ROUND-PAD -> JST-XH-03-PIN-ROUND-PAD; device Rembrandt Electronics - JST XH Connectors v1-0:JST-XH-02-PACKAGE-ROUND-PAD -> Rembrandt Electronics - JST XH Connectors v1-0:JST-XH-03-PACKAGE-ROUND-PAD
- moved X6 3.81 mm to (-33.1, 44.7)
- moved X5 3.81 mm to (-33.1, 35.7)
- moved X4 2.54 mm to (-33.0, 25.4)
Connections:
- net 3.3V: now also X4.1
- net A3: now also X4.3; no longer X4.2
- net GND: now also X4.2; no longer X4.1
Routing:
- net 3.3V: track 86.1 -> 102.6 mm
- net D4: track 26.3 -> 32.8 mm
- net D3: track 15.8 -> 20.9 mm
- net A3: track 5.77 -> 7.09 mm

Commit message: CLeaned up layout board
Changed lines of the file:
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@@
 <hole x="-23.6474" y="-1.2192" drill="0.35"/>
 <hole x="-25.4508" y="47.0916" drill="0.35"/>
-<hole x="-52.0954" y="49.7586" drill="0.35"/>
+<hole x="-52.0954" y="49.7586" drill="1"/>
 <hole x="-37.6174" y="27.9908" drill="0.35"/>
 </plain>

Commit message: Remote almost finish
Parts:
- removed CN1: SOCKET 1x2, adafruit:JST-PH-2-THM
- removed J1: FEMALE 1x2, SparkFun-Retired:1X02
- removed J2, J6: 455-1750-1-ND, SparkFun-Connectors:1X03
- removed J4: FEMALE 2x4, SparkFun-Connectors:2X4
- removed J5: FEMALE 2x3, SparkFun-Connectors:2X3
- removed X1: JST-XH-04-PIN-ROUND-PAD, Rembrandt Electronics - JST XH Connectors v1-0:JST-XH-04-PACKAGE-ROUND-PAD
- removed X2, X3, X5, X6: JST-XH-02-PIN-ROUND-PAD, Rembrandt Electronics - JST XH Connectors v1-0:JST-XH-02-PACKAGE-ROUND-PAD
- removed X4: JST-XH-03-PIN-ROUND-PAD, Rembrandt Electronics - JST XH Connectors v1-0:JST-XH-03-PACKAGE-ROUND-PAD
- added BATT: SOCKET 1x2, adafruit:JST-PH-2-THM
- added BUTTONS, CHARGE, HALL, LED: JST-XH-03-PIN-ROUND-PAD, Rembrandt Electronics - JST XH Connectors v1-0:JST-XH-03-PACKAGE-ROUND-PAD
- added NRF: FEMALE 2x4, SparkFun-Connectors:2X4
- added OLED: JST-XH-04-PIN-ROUND-PAD, Rembrandt Electronics - JST XH Connectors v1-0:JST-XH-04-PACKAGE-ROUND-PAD
- added PROG: FEMALE 2x3, SparkFun-Connectors:2X3
- added R10, R11, R9: 470, rcl:R0805
- added SW: 455-1750-1-ND, SparkFun-Connectors:1X03
- added USB: FEMALE 1x2, SparkFun-Retired:1X02
- moved R8 12.0 mm to (-30.8, 10.7), flipped to the bottom, turned to 180 degrees
- moved R7 10.7 mm to (-32.7, 13.6), flipped to the bottom, turned to 0 degrees
- moved R3 8.52 mm to (-44.5, -15.2), flipped to the bottom
- moved VR1 8.35 mm to (-24.8, -5.08)
- moved U1 6.56 mm to (-32.4, -5.08)
- moved R2 4.39 mm to (-40.1, 19.1), turned to 180 degrees
- moved C10 3.42 mm to (-35.6, -15.9)
- moved IC1 3.42 mm to (-31.8, -15.9)
- moved Q1 2.54 mm to (-35.6, -11.4)
- moved U2 2.54 mm to (-30.5, -11.4)
- moved U4 1.55 mm to (-31.8, 11.4)
- moved C1 1.42 mm to (-32.4, 1.27)
- moved C6 1.42 mm to (-43.8, 15.2)
- moved C7 1.42 mm to (-43.8, 10.2)
- moved R4 1.42 mm to (-23.5, -17.8)
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Connections:
- new net N$2: CHARGE.1, R9.2
- net 3.3V: now also HALL.1, NRF.2, OLED.2; no longer J4.2, X1.2, X4.1
- net A3: now also HALL.3; no longer X4.3
- net CE: now also NRF.3; no longer J4.3
- net CSN: now also NRF.4; no longer J4.4
- net D0: no longer J6.2
- net D1: no longer J6.3
- net D2: now also BUTTONS.1; no longer X3.2
- net D3: now also BUTTONS.2; no longer X5.2
- net D4: now also LED.1, R11.1; no longer X6.2
- net D5: now also LED.2, R10.1
- net GND: now also BATT.2, BUTTONS.3, HALL.2, LED.3, NRF.1, OLED.1, PROG.6, R10.2, R11.2, R9.1, USB.1; no longer CN1.1, J1.1, J4.1, J5.6, J6.1, X1.1, X3.1, X4.2, X5.1, X6.1
- net MISO: now also NRF.7, PROG.1; no longer J4.7, J5.1
- net MOSI: now also NRF.6, PROG.4; no longer J4.6, J5.4
- net N$10: now also BATT.1, SW.2; no longer CN1.2, J2.2
- net N$5: now also CHARGE.2; no longer X2.1
- net RST: now also PROG.5; no longer J5.5
- net SCK: now also NRF.5, PROG.3; no longer J4.5, J5.3
- net SCL: now also OLED.3; no longer X1.3
- net SDA: now also OLED.4; no longer X1.4
- net V_BATT: now also SW.1; no longer J2.1
- net V_USB: now also CHARGE.3, USB.2; no longer J1.2, X2.2
Routing:
- net D5: track 0.00 -> 44.4 mm, vias 0 -> 1
- net VIN: track 62.7 -> 45.8 mm
- net GND: track 9.45 -> 24.0 mm, vias 4 -> 7
- net A3: track 7.09 -> 19.6 mm, vias 1 -> 0
- net D1: track 12.1 -> 0.00 mm
- net V_BATT: track 69.6 -> 58.0 mm, vias 2 -> 3
- net D2: track 24.1 -> 13.4 mm, vias 1 -> 0
- net D0: track 10.2 -> 0.00 mm
- net N$5: track 13.1 -> 3.20 mm
- net N$4: track 5.82 -> 13.5 mm, vias 0 -> 1
- net MISO: track 18.4 -> 25.2 mm
- net A2: track 14.9 -> 8.60 mm, vias 0 -> 1
- net N$1: track 4.40 -> 10.6 mm
- net MOSI: track 22.0 -> 27.6 mm
- net STATUS: track 9.35 -> 3.84 mm
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Other:
- board text removed: "BATT"
- board text removed: "CHRG LED"
- board text removed: "DEADMAN"
- board text removed: "HALL"
- board text removed: "MAIN SWITCH"
- board text removed: "MP BUTTON"
- board text removed: "NRF"
- board text removed: "OLED"
- board text removed: "PROG"
- board text removed: "RX"
- board text removed: "TX"
- board text removed: "UART"
- board text removed: "USB PWR"

Commit message: PCB DOne
Routing:
- net GND: track 24.0 -> 32.7 mm, vias 7 -> 11
- net V_BATT: track 58.0 -> 56.6 mm
- net SCK: track 26.3 -> 27.6 mm
Changed lines of the file:
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@@
 <wire x1="-23.495" y1="11.4554" x2="-25.5778" y2="9.3726" width="0.254" layer="16"/>
 <wire x1="-25.5778" y1="9.3726" x2="-25.5778" y2="6.0452" width="0.254" layer="16"/>
-<wire x1="-35.56" y1="-14.925" x2="-44.45" y2="-19.37" width="0" layer="19" extent="1-16"/>
-<wire x1="-32.385" y1="0.32" x2="-30.48635" y2="1.27" width="0" layer="19" extent="1-1"/>
-<wire x1="-25.5778" y1="6.0452" x2="-25.4" y2="3.49" width="0" layer="19" extent="1-1"/>
-<wire x1="-36.04396875" y1="11.044984375" x2="-36.038384375" y2="12.644975" width="0" layer="19" extent="1-1"/>
+<via x="-37.211" y="12.7762" extent="1-16" drill="0.35"/>
+<via x="-38.6842" y="11.7602" extent="1-16" drill="0.35"/>
+<via x="-40.005" y="14.4018" extent="1-16" drill="0.35"/>
+<wire x1="-37.211" y1="12.7762" x2="-38.227" y2="11.7602" width="0.254" layer="16"/>
+<wire x1="-38.227" y1="11.7602" x2="-38.6842" y2="11.7602" width="0.254" layer="16"/>
+<wire x1="-38.6842" y1="11.7602" x2="-40.005" y2="13.081" width="0.254" layer="16"/>
+<wire x1="-40.005" y1="13.081" x2="-40.005" y2="14.4018" width="0.254" layer="16"/>
+<wire x1="-32.385" y1="0.32" x2="-31.435" y2="1.27" width="0.254" layer="1"/>
+<wire x1="-31.435" y1="1.27" x2="-30.48635" y2="1.27" width="0.254" layer="1"/>
+<via x="-44.45" y="-18.0848" extent="1-16" drill="0.35"/>
+<wire x1="-44.45" y1="-18.0848" x2="-44.45" y2="-19.37" width="0.254" layer="16"/>
 </signal>
 <signal name="V_BATT">
@@
 <wire x1="-36.86" y1="-11.43" x2="-36.86" y2="-10.48" width="0.254" layer="1"/>
 <wire x1="-34.26" y1="-10.48" x2="-36.86" y2="-10.48" width="0.254" layer="1"/>
-<wire x1="-33.26826875" y1="-13.4366" x2="-37.5158" y2="-13.4366" width="0.254" layer="1"/>
-<wire x1="-37.5158" y1="-13.4366" x2="-37.5158" y2="-12.96933125" width="0.254" layer="1"/>
-<wire x1="-37.5158" y1="-12.96933125" x2="-37.6394" y2="-12.84573125" width="0.254" layer="1"/>
-<wire x1="-37.6394" y1="-12.84573125" x2="-37.6394" y2="-11.91426875" width="0.254" layer="1"/>
-<wire x1="-37.6394" y1="-11.91426875" x2="-37.47573125" y2="-11.7506" width="0.254" layer="1"/>
-<wire x1="-37.47573125" y1="-11.7506" x2="-37.1806" y2="-11.7506" width="0.254" layer="1"/>
-<wire x1="-37.1806" y1="-11.7506" x2="-36.86" y2="-11.43" width="0.254" layer="1"/>
+<wire x1="-33.26826875" y1="-13.4366" x2="-37.6394" y2="-13.4366" width="0.254" layer="1"/>
+<wire x1="-37.6394" y1="-13.4366" x2="-37.6394" y2="-11.91426875" width="0.254" layer="1"/>
+<wire x1="-37.6394" y1="-11.91426875" x2="-37.17093125" y2="-11.4458" width="0.254" layer="1"/>
+<wire x1="-37.17093125" y1="-11.4458" x2="-36.8758" y2="-11.4458" width="0.254" layer="1"/>
+<wire x1="-36.8758" y1="-11.4458" x2="-36.86" y2="-11.43" width="0.254" layer="1"/>
 <wire x1="-31.7642" y1="-14.94066875" x2="-33.26826875" y2="-13.4366" width="0.254" layer="1"/>
 <wire x1="-34.26" y1="-10.48" x2="-31.79445" y2="-10.48" width="0.254" layer="1"/>
@@
 <wire x1="-33.909" y1="11.43" x2="-33.909" y2="13.396" width="0.254" layer="16"/>
 <wire x1="-33.909" y1="13.396" x2="-33.6906" y2="13.6144" width="0.254" layer="16"/>
-<wire x1="-36.6522" y1="-8.255" x2="-35.56" y2="-7.1628" width="0.254" layer="16"/>
 <via x="-34.4932" y="2.286" extent="1-16" drill="0.35"/>
 <wire x1="-36.6522" y1="-8.255" x2="-36.6522" y2="-1.5464125" width="0.254" layer="1"/>
@@
 <wire x1="-27.9908" y1="-18.73" x2="-29.8958" y2="-16.825" width="0.254" layer="1"/>
 <wire x1="-27.9908" y1="-18.73" x2="-26.67" y2="-18.73" width="0.254" layer="1"/>
-<wire x1="-41.91" y1="-15.24" x2="-40.83775" y2="-15.24" width="0.254" layer="16"/>
+<wire x1="-41.32035" y1="-15.24" x2="-41.91" y2="-15.24" width="0.254" layer="16"/>
 <wire x1="-34.53459375" y1="-16.4564" x2="-28.661396875" y2="-22.329596875" width="0.254" layer="16"/>
-<wire x1="-40.83775" y1="-15.24" x2="-39.62135" y2="-16.4564" width="0.254" layer="16"/>
-<wire x1="-39.62135" y1="-16.4564" x2="-34.53459375" y2="-16.4564" width="0.254" layer="16"/>
+<wire x1="-34.53459375" y1="-16.4564" x2="-36.83" y2="-16.4564" width="0.254" layer="16"/>
+<wire x1="-36.83" y1="-16.4564" x2="-40.10395" y2="-16.4564" width="0.254" layer="16"/>
 <wire x1="-31.3294" y1="-15.31573125" x2="-31.3294" y2="-14.53426875" width="0.254" layer="1"/>
 <wire x1="-31.3294" y1="-14.53426875" x2="-31.16573125" y2="-14.3706" width="0.254" layer="1"/>
@@
 <wire x1="-29.52546875" y1="-14.5794" x2="-24.1594" y2="-14.5794" width="0.254" layer="1"/>
 <wire x1="-24.1594" y1="-14.5794" x2="-24.13" y2="-14.55" width="0.254" layer="1"/>
+<wire x1="-40.10395" y1="-16.4564" x2="-41.32035" y2="-15.24" width="0.254" layer="16"/>
 </signal>
 <signal name="3.3V">
@@
 <wire x1="-33.5788" y1="1.27" x2="-27.5082" y2="7.3406" width="0.254" layer="16"/>
 <wire x1="-38.1" y1="1.27" x2="-33.5788" y2="1.27" width="0.254" layer="16"/>
-<wire x1="-27.467196875" y1="8.61503125" x2="-27.5082" y2="7.3406" width="0" layer="19" extent="1-1"/>
+<wire x1="-27.5082" y1="7.3406" x2="-27.5082" y2="8.574028125" width="0.254" layer="1"/>
+<wire x1="-27.5082" y1="8.574028125" x2="-27.467196875" y2="8.61503125" width="0.254" layer="1"/>
 </signal>
 <signal name="MOSI">
