File: eagle/board/pcbboard.brd (EAGLE design)
At the start: 70.5 x 43.2 mm, 40 parts, among them U2 ATMEGA328P-PU, Y2 16MHz

Commit message: Remote almost finish
Parts:
- removed C6: .1u, rcl:C0805
- added 3.3V, 5V: (no value), adafruit:LED3MM
- added C1: .1u, rcl:C0805
- added R12, R2: 470, rcl:R0805
- added RX_EN, TX_EN: (no value), SparkFun-Connectors:1X02
- R10, R11: value 470 -> 10k
- R7, R8: value 10k -> 470
- moved R7 25.5 mm to (31.8, 13.3)
- moved R6 21.6 mm to (29.2, 13.3)
- moved R10 21.6 mm to (10.8, 27.9), turned to 90 degrees
- moved R5 21.1 mm to (14.0, 27.9)
- moved R8 19.4 mm to (26.7, 13.3)
- moved R11 16.5 mm to (7.62, 13.3), turned to 90 degrees
- moved C2 15.5 mm to (19.1, 27.9), turned to 90 degrees
- moved C3 9.92 mm to (11.4, 21.6), turned to 0 degrees
- moved R9 7.62 mm to (24.1, 13.3)
- moved TP_H1-2 5.75 mm to (-7.62, 3.17)
- moved TP_H2-2 4.95 mm to (12.7, 3.94)
- moved TP_3.3V 3.81 mm to (-6.99, 14.6)
- moved TP_5V 3.81 mm to (-11.4, 14.6)
- moved TP_H1-1 2.01 mm to (-7.62, -0.64)
- moved TP_H2-1 1.27 mm to (12.7, 0.00)
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- renumbered U$1 to X3, U$2 to X2, U2 to U1, Y2 to Y1
Connections:
- new net N$10: RX_EN.1, U1.2
- new net N$11: TX_EN.1, U1.3
- new net N$6: 3.3V.K, R2.1
- new net N$7: 5V.K, R12.1
- net +5V: now also 5V.A, C1.1, R10.1, R11.1; no longer C3.1, R7.1, R8.1
- net 3.3V: now also 3.3V.A
- net A0: now also R5.2; no longer R8.2
- net A1: now also R10.2; no longer R7.2
- net AREF: now also C3.1; no longer C6.1
- net D3: now also R11.2; no longer R6.2
- net D5: now also R9.1; no longer R11.1
- net D6: now also R8.1; no longer R10.1
- net D7: now also R6.2; no longer R5.2
- net D8: now also R7.1; no longer R9.1
- net GND: now also C1.2, R12.2, R2.2; no longer C6.2
- net N$2: now also R7.2; no longer R9.2
- net N$3: now also R8.2; no longer R10.2
- net N$4: now also R9.2; no longer R11.2
- net RX: now also RX_EN.2; no longer U1.2
- net TX: now also TX_EN.2; no longer U1.3
Routing:
- net +5V: track 0.00 -> 215.1 mm
- net 3.3V: track 0.00 -> 73.6 mm, vias 0 -> 2
- net RST: track 0.00 -> 56.3 mm
- net SCK: track 0.00 -> 43.7 mm
- net MISO: track 0.00 -> 38.6 mm
- net D7: track 0.00 -> 38.3 mm
- net MOSI: track 0.00 -> 38.1 mm
- net D4: track 0.00 -> 28.9 mm
- net D6: track 0.00 -> 28.6 mm
- net D3: track 0.00 -> 27.3 mm
- net D5: track 0.00 -> 26.1 mm
- net A0: track 0.00 -> 24.4 mm
- net D2: track 0.00 -> 23.8 mm
- net CSN: track 0.00 -> 17.0 mm
- net A1: track 0.00 -> 17.0 mm
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